File: Voltmeter/Voltmeter.sch (KiCad schematic (older format))
At the start: 45 parts, among them J1 Input 1, J10 Input 10, J11 Input 11, J2 Input 2, J3 Input 3, J4 Input 4, J5 Input 5, J6 Input 6, J7 Input 7, J8 Input 8, J9 Input 9, U1 CD74HC4067M, U1 LM35-LP, U1 LM7805_TO220

Commit message: my commit
Parts:
- removed R15: 39k, symbol Device:R_Small_US
- removed R16: 8.2k, symbol Device:R_Small_US
- added U4: LCD_I2C, kicad-library:LCD_I2C, symbol Lcd_I2C:LCD_I2C
- C1: value C_Small -> .33uF; footprint (none) -> Capacitor_THT:C_Disc_D3.4mm_W2.1mm_P2.50mm
- C2: value C_Small -> .1uF; footprint (none) -> Capacitor_THT:C_Disc_D3.4mm_W2.1mm_P2.50mm
- D1: renamed from D0; value D_Zener_4.9V -> D_Zener_5.1V; footprint (none) -> Resistor_THT:R_Axial_DIN0207_L6.3mm_D2.5mm_P7.62mm_Horizontal
- J1, J10, J11, J2, J3, J4, J5, J6, J7, J8, J9: footprint (none) -> kicad-library:TerminalBlock_Altech_AK300-2_P5.00mm
- J_INP1: renamed from J_INP; footprint (none) -> kicad-library:TerminalBlock_Altech_AK300-2_P5.00mm
- R1: renamed from R23; footprint (none) -> Resistor_THT:R_Axial_DIN0207_L6.3mm_D2.5mm_P7.62mm_Horizontal
- R10: renamed from R6; footprint (none) -> Resistor_THT:R_Axial_DIN0207_L6.3mm_D2.5mm_P7.62mm_Horizontal
- R11: renamed from R7; footprint (none) -> Resistor_THT:R_Axial_DIN0207_L6.3mm_D2.5mm_P7.62mm_Horizontal
- R12: renamed from R8; footprint (none) -> Resistor_THT:R_Axial_DIN0207_L6.3mm_D2.5mm_P7.62mm_Horizontal
- R13: renamed from R9; footprint (none) -> Resistor_THT:R_Axial_DIN0207_L6.3mm_D2.5mm_P7.62mm_Horizontal
- R14: renamed from R10; footprint (none) -> Resistor_THT:R_Axial_DIN0207_L6.3mm_D2.5mm_P7.62mm_Horizontal
- R15: renamed from R11; footprint (none) -> Resistor_THT:R_Axial_DIN0207_L6.3mm_D2.5mm_P7.62mm_Horizontal
- R16: renamed from R12; footprint (none) -> Resistor_THT:R_Axial_DIN0207_L6.3mm_D2.5mm_P7.62mm_Horizontal
- R17: renamed from R13; footprint (none) -> Resistor_THT:R_Axial_DIN0207_L6.3mm_D2.5mm_P7.62mm_Horizontal
- R18: renamed from R14; footprint (none) -> Resistor_THT:R_Axial_DIN0207_L6.3mm_D2.5mm_P7.62mm_Horizontal
- R2: renamed from R24; footprint (none) -> Resistor_THT:R_Axial_DIN0207_L6.3mm_D2.5mm_P7.62mm_Horizontal
- R21: renamed from R17; footprint (none) -> Resistor_THT:R_Axial_DIN0207_L6.3mm_D2.5mm_P7.62mm_Horizontal
- R22: renamed from R18; footprint (none) -> Resistor_THT:R_Axial_DIN0207_L6.3mm_D2.5mm_P7.62mm_Horizontal
- R23: renamed from R19; footprint (none) -> Resistor_THT:R_Axial_DIN0207_L6.3mm_D2.5mm_P7.62mm_Horizontal
- R24: renamed from R20; footprint (none) -> Resistor_THT:R_Axial_DIN0207_L6.3mm_D2.5mm_P7.62mm_Horizontal
- R25: renamed from R21; footprint (none) -> Resistor_THT:R_Axial_DIN0207_L6.3mm_D2.5mm_P7.62mm_Horizontal
- R26: renamed from R22; footprint (none) -> Resistor_THT:R_Axial_DIN0207_L6.3mm_D2.5mm_P7.62mm_Horizontal
- R3: renamed from R25; footprint (none) -> Resistor_THT:R_Axial_DIN0207_L6.3mm_D2.5mm_P7.62mm_Horizontal
- R4: renamed from R26; footprint (none) -> Resistor_THT:R_Axial_DIN0207_L6.3mm_D2.5mm_P7.62mm_Horizontal
- R5: renamed from R1; footprint (none) -> Resistor_THT:R_Axial_DIN0207_L6.3mm_D2.5mm_P7.62mm_Horizontal
- R6: renamed from R2; footprint (none) -> Resistor_THT:R_Axial_DIN0207_L6.3mm_D2.5mm_P7.62mm_Horizontal
- R7: renamed from R3; footprint (none) -> Resistor_THT:R_Axial_DIN0207_L6.3mm_D2.5mm_P7.62mm_Horizontal
- R8: renamed from R4; footprint (none) -> Resistor_THT:R_Axial_DIN0207_L6.3mm_D2.5mm_P7.62mm_Horizontal
- R9: renamed from R5; footprint (none) -> Resistor_THT:R_Axial_DIN0207_L6.3mm_D2.5mm_P7.62mm_Horizontal
- U2: renamed from U1; footprint (none) -> Package_TO_SOT_THT:TO-92L_HandSolder
- U3: renamed from U1; footprint Package_SO:SOIC-24W_7.5x15.4mm_P1.27mm -> kicad-library:74hc4067_Breakout
Connections:
- net +5V: now also U4.1 (VCC)
- net D10: now also U3.11 (S1); no longer U3.14 (S2)
- net D11: now also U3.10 (S0); no longer U3.13 (S3)
- net D8: now also U3.13 (S3); no longer U3.10 (S0)
- net D9: now also U3.14 (S2); no longer U3.11 (S1)
- net GND: now also U4.2 (GND)
- net SDA: now reaches A1.23 (A4)
- net SDA: now also U4.3 (SDA)
- net SCL: now reaches A1.24 (A5)
- net SCL: now also U4.4 (SCL)
